File: PCB/mcu/digiobscura_mcu.sch (KiCad schematic (older format))
At the start: 45 parts, among them J1 Conn_01x02, J11 Conn_01x08, J2 ROW, J3 COL, J4 Micro_SD_Card_Det, P1 USB_OTG, P2 CONN_01X07, SW1 SW_Push_SPDT, SW2 SW_Push, U1 SAMD21G18A_ArduinoSimple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

Commit message: Fixed BOM
Parts:
- D1: Digikey Part No. (none) -> 1080-1403-2-ND
- J1: Digikey Part No. (none) -> 455-1719-ND
- J11: Digikey Part No. (none) -> S7041-ND
- J2, J3: Digikey Part No. (none) -> S7044-ND
- RV1: Digikey Part No. (none) -> 987-1276-ND
- SW1: Digikey Part No. (none) -> CKN9542-ND
- SW2: Digikey Part No. (none) -> P12961SCT-ND
- U1: Digikey Part No. (none) -> ATSAMD21G18A-AUTCT-ND
Changed lines of the file:
@@
 F 2 "Connector_PinSocket_2.54mm:PinSocket_1x08_P2.54mm_Vertical" H 7050 2800 50  0001 C CNN
 F 3 "~" H 7050 2800 50  0001 C CNN
+F 4 "S7041-ND" H 7050 2800 50  0001 C CNN "Digikey Part No."
 	1    7050 2800
 	-1   0    0    -1
@@
 F 2 "Package_QFP:LQFP-48_7x7mm_P0.5mm" H 4025 5311 32  0000 C CIN
 F 3 "" H 3950 3900 60  0000 C CNN
+F 4 "ATSAMD21G18A-AUTCT-ND" H 3950 3650 50  0001 C CNN "Digikey Part No."
 	1    3950 3650
 	1    0    0    -1
@@
 F 2 "Connector_PinSocket_2.54mm:PinSocket_1x11_P2.54mm_Vertical" H 11900 7650 50  0001 C CNN
 F 3 "~" H 11900 7650 50  0001 C CNN
+F 4 "S7044-ND" H 11900 7650 50  0001 C CNN "Digikey Part No."
 	1    11900 7650
 	1    0    0    -1
@@
 F 2 "LED_SMD:LED_0603_1608Metric" V 10700 1700 50  0001 C CNN
 F 3 "" V 10700 1700 50  0001 C CNN
+F 4 "1080-1403-2-ND" H 10700 1700 50  0001 C CNN "Digikey Part No."
 	1    10700 1700
 	0    -1   -1   0
@@
 F 2 "Connector_JST:JST_PH_S2B-PH-K_1x02_P2.00mm_Horizontal" H 10800 5500 50  0001 C CNN
 F 3 "~" H 10800 5500 50  0001 C CNN
+F 4 "455-1719-ND" H 10800 5500 50  0001 C CNN "Digikey Part No."
 	1    10800 5500
 	1    0    0    -1
@@
 F 2 "Potentiometer_THT:Potentiometer_Bourns_PTV09A-1_Single_Vertical" H 13800 7350 50  0001 C CNN
 F 3 "~" H 13800 7350 50  0001 C CNN
+F 4 "987-1276-ND" H 13800 7350 50  0001 C CNN "Digikey Part No."
 	1    13800 7350
 	0    -1   -1   0
@@
 F 2 "Connector_PinSocket_2.54mm:PinSocket_1x11_P2.54mm_Vertical" H 15200 7600 50  0001 C CNN
 F 3 "~" H 15200 7600 50  0001 C CNN
+F 4 "S7044-ND" H 15200 7600 50  0001 C CNN "Digikey Part No."
 	1    15200 7600
 	1    0    0    -1
@@
 F 2 "Button_Switch_THT:SW_Slide_1P2T_CK_OS102011MS2Q" H 1650 7900 50  0001 C CNN
 F 3 "~" H 1650 7900 50  0001 C CNN
+F 4 "CKN9542-ND" H 1650 7900 50  0001 C CNN "Digikey Part No."
 	1    1650 7900
 	1    0    0    -1
@@
 F 2 "Button_Switch_SMD:SW_SPST_EVPBF" H 12800 5750 50  0001 C CNN
 F 3 "~" H 12800 5750 50  0001 C CNN
+F 4 "P12961SCT-ND" H 12800 5550 50  0001 C CNN "Digikey Part No."
 	1    12800 5550
 	1    0    0    -1
