File: PCB/image_sensor/digiobscura.sch (KiCad schematic (older format))
At the start: 1032 parts, among them J1 ROW, J2 COL, Q1 ALS-PT19, Q10 ALS-PT19, Q100 ALS-PT19, Q1000 ALS-PT19, Q1001 ALS-PT19, Q1002 ALS-PT19, Q1003 ALS-PT19, Q1004 ALS-PT19, Q1005 ALS-PT19, Q1006 ALS-PT19, Q1007 ALS-PT19, Q1008 ALS-PT19, Q1009 ALS-PT19, Q101 ALS-PT19, Q1010 ALS-PT19, Q1011 ALS-PT19, Q1012 ALS-PT19, Q1013 ALS-PT19, Q1014 ALS-PT19, Q1015 ALS-PT19, Q1016 ALS-PT19, Q1017 ALS-PT19, Q1018 ALS-PT19, Q1019 ALS-PT19, Q102 ALS-PT19, Q1020 ALS-PT19, Q1021 ALS-PT19, Q1022 ALS-PT19, Q1023 ALS-PT19, Q1024 ALS-PT19, Q103 ALS-PT19, Q104 ALS-PT19, Q105 ALS-PT19, Q106 ALS-PT19, Q107 ALS-PT19, Q108 ALS-PT19, Q109 ALS-PT19, Q11 ALS-PT19, Q110 ALS-PT19, Q111 ALS-PT19, Q112 ALS-PT19, Q113 ALS-PT19, Q114 ALS-PT19, Q115 ALS-PT19, Q116 ALS-PT19, Q117 ALS-PT19, Q118 ALS-PT19, Q119 ALS-PT19, Q12 ALS-PT19, Q120 ALS-PT19, Q121 ALS-PT19, Q122 ALS-PT19, Q123 ALS-PT19, Q124 ALS-PT19, Q125 ALS-PT19, Q126 ALS-PT19, Q127 ALS-PT19, Q128 ALS-PT19, Q129 ALS-PT19, Q13 ALS-PT19, Q130 ALS-PT19, Q131 ALS-PT19, Q132 ALS-PT19, Q133 ALS-PT19, Q134 ALS-PT19, Q135 ALS-PT19, Q136 ALS-PT19, Q137 ALS-PT19, Q138 ALS-PT19, Q139 ALS-PT19, Q14 ALS-PT19, Q140 ALS-PT19, Q141 ALS-PT19, Q142 ALS-PT19, Q143 ALS-PT19, Q144 ALS-PT19, Q145 ALS-PT19, Q146 ALS-PT19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

Commit message: updated BOM files
Parts:
- J1, J2: Digikey Part No. S7044-ND -> 609-5133-ND
Changed lines of the file:
@@
 F 2 "Connector_PinHeader_2.54mm:PinHeader_1x11_P2.54mm_Vertical" H 30800 12200 50  0001 C CNN
 F 3 "~" H 30800 12200 50  0001 C CNN
-F 4 "S7044-ND" H 30800 12200 50  0001 C CNN "Digikey Part No."
+F 4 "609-5133-ND" H 30800 12200 50  0001 C CNN "Digikey Part No."
 	1    30800 12200
 	1    0    0    -1
@@
 F 2 "Connector_PinHeader_2.54mm:PinHeader_1x11_P2.54mm_Vertical" H 34100 12150 50  0001 C CNN
 F 3 "~" H 34100 12150 50  0001 C CNN
-F 4 "S7044-ND" H 34100 12150 50  0001 C CNN "Digikey Part No."
+F 4 "609-5133-ND" H 34100 12150 50  0001 C CNN "Digikey Part No."
 	1    34100 12150
 	1    0    0    -1
